Commit message: ..

File: project/assets/labyr2t.urdf (robot description, URDF)
Before this commit: robot labyr2t, 16 links, 15 joints
Links:
- added link EnteringWall_link, mass 1.00000; collision box size=0.10000 2.00000 2.00000; visual box size=0.10000 2.00000 2.00000
Joints:
- added joint EnteringWall_link_joint: type fixed, parent floor_link, child EnteringWall_link, origin xyz=2.95000 0.00000 1.05000 rpy=0.00000 0.00000 0.00000

Commit message: Labirinti aggiornati

File: project/assets/labyr2t.urdf (robot description, URDF)
Before this commit: robot labyr2t, 17 links, 16 joints
Links:
- link floor_link: geometry collision box size=6.00000 10.40000 0.10000; visual box size=6.00000 10.40000 0.10000
- link wall10_link: geometry collision box size=0.10000 2.00000 2.00000; visual box size=0.10000 2.00000 2.00000
- link wall12_link: geometry collision box size=0.10000 2.00000 2.00000; visual box size=0.10000 2.00000 2.00000
- link wall4_link: geometry collision box size=0.10000 2.00000 2.00000; visual box size=0.10000 2.00000 2.00000
- link wall6_link: geometry collision box size=0.10000 2.00000 2.00000; visual box size=0.10000 2.00000 2.00000
Joints:
- joint wall10_link_joint: origin xyz=-2.95000 -4.00000 1.05000 rpy=0.00000 0.00000 0.00000 -> xyz=-2.95000 -4.10000 1.05000 rpy=0.00000 0.00000 0.00000
- joint wall11_link_joint: origin xyz=0.00000 -4.95000 1.05000 rpy=0.00000 0.00000 0.00000 -> xyz=0.00000 -5.15000 1.05000 rpy=0.00000 0.00000 0.00000
- joint wall12_link_joint: origin xyz=2.95000 -4.00000 1.05000 rpy=0.00000 0.00000 0.00000 -> xyz=2.95000 -4.10000 1.05000 rpy=0.00000 0.00000 0.00000
- joint wall4_link_joint: origin xyz=2.95000 4.00000 1.05000 rpy=0.00000 0.00000 0.00000 -> xyz=2.95000 4.10000 1.05000 rpy=0.00000 0.00000 0.00000
- joint wall5_link_joint: origin xyz=0.00000 4.95000 1.05000 rpy=0.00000 0.00000 0.00000 -> xyz=0.00000 5.15000 1.05000 rpy=0.00000 0.00000 0.00000

File: project/assets/labyr2t_v2.urdf (robot description, URDF)
Before this commit: robot labyr2t_v2, 16 links, 15 joints
Links:
- added link EnteringWall_link, mass 1.00000; collision box size=0.20000 2.00000 2.00000; visual box size=0.20000 2.00000 2.00000
- link floor_link: geometry collision box size=12.00000 20.40000 0.10000; visual box size=12.00000 20.40000 0.10000
- link wall10_link: geometry collision box size=0.20000 2.00000 2.00000; visual box size=0.20000 2.00000 2.00000
- link wall12_link: geometry collision box size=0.20000 2.00000 2.00000; visual box size=0.20000 2.00000 2.00000
- link wall4_link: geometry collision box size=0.20000 2.00000 2.00000; visual box size=0.20000 2.00000 2.00000
- link wall6_link: geometry collision box size=0.20000 2.00000 2.00000; visual box size=0.20000 2.00000 2.00000
Joints:
- added joint EnteringWall_link_joint: type fixed, parent floor_link, child EnteringWall_link, origin xyz=5.90000 0.00000 1.05000 rpy=0.00000 0.00000 0.00000
- joint wall10_link_joint: origin xyz=-5.90000 -8.90000 1.05000 rpy=0.00000 0.00000 0.00000 -> xyz=-5.90000 -9.00000 1.05000 rpy=0.00000 0.00000 0.00000
- joint wall11_link_joint: origin xyz=0.00000 -9.90000 1.05000 rpy=0.00000 0.00000 0.00000 -> xyz=0.00000 -10.10000 1.05000 rpy=0.00000 0.00000 0.00000
- joint wall12_link_joint: origin xyz=5.90000 -8.90000 1.05000 rpy=0.00000 0.00000 0.00000 -> xyz=5.90000 -9.00000 1.05000 rpy=0.00000 0.00000 0.00000
- joint wall5_link_joint: origin xyz=0.00000 9.90000 1.05000 rpy=0.00000 0.00000 0.00000 -> xyz=0.00000 10.10000 1.05000 rpy=0.00000 0.00000 0.00000
- joint wall6_link_joint: origin xyz=-5.90000 8.90000 1.05000 rpy=0.00000 0.00000 0.00000 -> xyz=-5.90000 9.00000 1.05000 rpy=0.00000 0.00000 0.00000
